File: Hardware/CHAIRI2CXIAO.sch (EAGLE design)
At the start: 23 parts, among them IC1 DS3502, IC2 DS3502, J1 OUTPUT, J2 M06-PLAIN

Commit message: Major conversion to use ESP32 in UB5 plastic box.
Parts:
- removed C2: 100nF, SuperHouse-DiscreteSemi:CAP0603
- removed FID1, FID2: FIDUCIAL1X2.5, SuperHouse-Symbols:FIDUCIAL1X2.5
- removed LED1: BLUE, SuperHouse-LEDs:LED0603
- removed R4: 4K7, SuperHouse-DiscreteSemi:RESISTOR0603
- removed SJ1, SJ2: PU, SuperHouse-Jumpers:SJC-NORMAL
- added C4, C5, C6: 10uF, SuperHouse-DiscreteSemi:CAP0805
- added C7: 1uF, SuperHouse-DiscreteSemi:CAP0603
- added C8: 100nF, SuperHouse-DiscreteSemi:CAP0603
- added F1: 500mA 1812 PTC, SuperHouse-Fuses:PTC050
- added IC3: ESPWROOM32, SuperHouse-MCUs:ESPWROOM32
- added IC5: CP2102N-A01-GQFN24, SuperHouse-ICs:CP2104
- added J3: BUT5, SuperHouse-Connectors:M01-PLAIN
- added LED3: BLUE, SuperHouse-LEDs:LED0603
- added LED4: RX/GRN, SuperHouse-LEDs:LED0603
- added LED5: TX/YEL, SuperHouse-LEDs:LED0603
- added Q1: MMDT3904, SuperHouse-DiscreteSemi:TRANS_NPN_DUAL-MMDT3904
- added R14, R15: 10K, SuperHouse-DiscreteSemi:RESISTOR0603
- added R16: 5.1K, SuperHouse-DiscreteSemi:RESISTOR0603
- added R17, R18: 22K, SuperHouse-DiscreteSemi:RESISTOR0603
- added R19: 22.1K, SuperHouse-DiscreteSemi:RESISTOR0603
- added R20: 47.5K, SuperHouse-DiscreteSemi:RESISTOR0603
- added R21, R22: 1K, SuperHouse-DiscreteSemi:RESISTOR0603
- added S2: RESET, SuperHouse-Switches:TAC_SWITCH_2PINSMT
- added U$35, U$36, U$37: FIDUCIAL1X2, SuperHouse-Symbols:FIDUCIAL1X2
- added VR1: AP2112KSOT25, SuperHouse-Regulators:AP2112KSOT25
- added Z1, Z2: PGB1010603, SuperHouse-DiscreteSemi:TVS0603
- J2: value M06-PLAIN -> USB-C-16P-16P; device SuperHouse-Connectors:M06-PLAIN -> SuperHouse-Connectors:USB-C-16P-16P
- R5: value 4K7 -> 10K
- R6: value 4K7 -> 5.1K
Connections:
- removed net N$5: LED1.A, R4.1
- removed net VCC: C2.1, IC1.VCC, IC2.A0, IC2.VCC, J2.5, R4.2, SJ1.2, SJ2.2
- new net !RESET: C7.1, IC3.EN, Q1Q1.C, R17.2, S2.S
- new net 3.3V: C5.1, C6.1, C8.1, IC1.VCC, IC2.A0, IC2.VCC, IC3.3V3, IC5.REGIN, IC5.VDD, IC5.VIO, LED4.A, LED5.A, R17.1, R18.1, R5.2, VR1.VOUT
- new net 5V: C4.1, F1.2, R19.2, VR1.EN, VR1.VIN
- new net D+: IC5.D+, J2.D+, Z2.2
- new net D-: IC5.D-, J2.D-, Z1.2
- new net DTR: IC5.DTR, Q1Q2.E, R14.1
- new net GPIO0: IC3.IO0, Q1Q2.C, R18.2
- new net N$10: J2.CC2, R16.2
- new net N$11: J2.CC1, R6.2
- new net N$13: LED5.C, R22.2
- new net N$39: IC5.VBUS, R19.1, R20.2
- new net N$7: Q1Q1.B, R14.2
- new net N$9: LED4.C, R21.2
- new net RTS: IC5.RTS, Q1Q1.E, R15.1
- new net RXD0: IC3.RXD0, IC5.TXD
- new net RX_LED: IC5.GPIO_1, R21.1
- new net TXD0: IC3.TXD0, IC5.RXD
- new net TX_LED: IC5.GPIO_0, R22.1
- new net VIN: F1.1, J2.VBUS
- net 12V: no longer J2.6
- net BUT5: now also J3.1; no longer J2.1
- net GND: now also C4.2, C5.2, C6.2, C7.2, C8.2, IC3.GND@1, IC3.GND@2, IC3.GND@3, IC3.GND@4, IC5.GND, IC5.GND_PAD, J2.GND, LED3.C, R16.1, R20.1, R6.1, S2.P, VR1.GND, Z1.1, Z2.1; no longer C2.2, J2.2, LED1.C
- net N$1: now also LED3.A, R5.1; no longer R5.2, SJ1.1
- net N$8: now also Q1Q2.B, R15.2; no longer R6.2, SJ2.1
- net SCL: now also IC3.IO22; no longer J2.4, R5.1
- net SDA: now also IC3.IO21; no longer J2.3, R6.1
Other:
- note added: "(C)2021 SuperHouse Automation: www.superhouse.tv"
- note added: "3.3V Power Supply"
- note added: "Auto Reset"
- note added: "Chair Power"
- note added: "ESP32 Microcontroller"
- note added: "GPIO0: GPIO1: USB_TX GPIO2: GPIO3: USB_RX GPIO4: GPIO13: GPIO16: GPIO17: GPIO18: GPIO21: SDA GPIO22: SCL GPIO23: GPIO25: GPIO27: Firmware: https://github.com/XXXXXX"
- note added: "Permobil Wheelchair Controller"
- note added: "SKU: PWC"
- note added: "USB-C Connection"
- note added: "USB-Serial Converter"
- note added: "V1.0 (2021-05-12)"
- note added: "WARNING: GPIO32/33 are used by RTC. Need to modify WROOM32 to use them as outputs"
- note added: "www.superhouse.tv/pwc"
- note removed: "(C)2020 SuperHouse Automation: www.superhouse.tv"
- note removed: "Chair Control I2C Interface"
- note removed: "I2C Interface"
- note removed: "Power Indicators"
- note removed: "SKU: CHAIRI2C"
- note removed: "V1.0 (2020-05-05)"
- note removed: "www.superhouse.tv/chairi2c"
